Commit message: changed names of links in URDF

File: src/arm/description/urdf/1000-Reduced Modelv6.urdf (robot description, URDF)
Before this commit: robot 1000-Reduced Modelv6, 7 links, 6 joints
Links:
- removed link base
- removed link bicep
- removed link forearm
- removed link shoulder
- removed link wrist pitch
- removed link wrist roll
- removed link wrist yaw
- added link base_link, mass 2.98521046700997; collision mesh filename=package://arm/description/meshes/base.STL; visual mesh filename=package://arm/description/meshes/base.STL
- added link bicep_link, mass 4.21157397014607; collision mesh filename=package://arm/description/meshes/bicep.STL; visual mesh filename=package://arm/description/meshes/bicep.STL
- added link forearm_link, mass 4.35871818699448; collision mesh filename=package://arm/description/meshes/forearm.STL; visual mesh filename=package://arm/description/meshes/forearm.STL
- added link shoulder_link, mass 4.54258438464217; collision mesh filename=package://arm/description/meshes/shoulder.STL; visual mesh filename=package://arm/description/meshes/shoulder.STL
- added link wrist_pitch_link, mass 0.86236150071068; collision mesh filename=package://arm/description/meshes/wrist pitch.STL; visual mesh filename=package://arm/description/meshes/wrist pitch.STL
- added link wrist_roll_link, mass 0.578594077815313; collision mesh filename=package://arm/description/meshes/wrist roll.STL; visual mesh filename=package://arm/description/meshes/wrist roll.STL
- added link wrist_yaw_link, mass 0.358868673438875; collision mesh filename=package://arm/description/meshes/wrist yaw.STL; visual mesh filename=package://arm/description/meshes/wrist yaw.STL
Joints:
- removed joint Base Yaw
- removed joint elbow pitch
- removed joint shoulder pitch
- removed joint wrist pitch
- removed joint wrist roll
- removed joint wrist yaw
- added joint base_yaw_joint: type revolute, parent base_link, child shoulder_link, origin xyz=-0.0420894636209815 -0.0119616169931191 0.0182598424192986 rpy=1.5707963267949 0 1.05545161052463, axis 0 1 0, limit lower=0 upper=0 effort=0 velocity=0
- added joint elbow_pitch_joint: type revolute, parent bicep_link, child forearm_link, origin xyz=0.0030875 0 -0.58189 rpy=0.51635 0 3.1416, axis -1 0 0, limit lower=0 upper=0 effort=0 velocity=0
- added joint shoulder_pitch_joint: type revolute, parent shoulder_link, child bicep_link, origin xyz=-0.0357971138440272 0.108175 0.00906194434350591 rpy=2.47061567686307 0.515344716270268 0, axis -1 0 0, limit lower=0 upper=0 effort=0 velocity=0
- added joint wrist_pitch_joint: type revolute, parent forearm_link, child wrist_pitch_link, origin xyz=0 0 0.581887499995086 rpy=1.29896997033974 -0.262305000585875 2.39226953786024, axis -0.707106781186547 0 0.707106781186548, limit lower=0 upper=0 effort=0 velocity=0
- added joint wrist_roll_joint: type revolute, parent wrist_yaw_link, child wrist_roll_link, origin xyz=0.00632947155943084 0.272267270409697 0.1004658595574 rpy=-1.56931940382504 -0.827547058181322 3.13950582346102, axis 0.000668221963468187 0.0176603835099617 -0.999843819970743, limit lower=0 upper=0 effort=0 velocity=0
- added joint wrist_yaw_joint: type revolute, parent wrist_pitch_link, child wrist_yaw_link, origin xyz=0.017777291445819 0 -0.017777291445819 rpy=-0.96359754736019 0.518498041049501 0.951194425773634, axis 0.706887306729703 0.0176165407866436 0.707106776289932, limit lower=0 upper=0 effort=0 velocity=0
