Commit message: launch file. Gazebo integration not working

File: src/arm/description/urdf/arm.xacro.urdf (robot description, URDF)
Before this commit: robot arm, 7 links, 6 joints
Links:
- added link dummy
Joints:
- added joint dummy_joint: type fixed, parent dummy, child base_link
- joint base_yaw_joint: limit lower=0 upper=0 effort=0 velocity=0 -> lower=-3.141592653589793 upper=3.141592653589793 effort=1000.0 velocity=2.5
- joint elbow_pitch_joint: limit lower=0 upper=0 effort=0 velocity=0 -> lower=-3.141592653589793 upper=3.141592653589793 effort=1000.0 velocity=2.5
- joint shoulder_pitch_joint: limit lower=0 upper=0 effort=0 velocity=0 -> lower=-3.141592653589793 upper=3.141592653589793 effort=1000.0 velocity=2.5
- joint wrist_pitch_joint: limit lower=0 upper=0 effort=0 velocity=0 -> lower=-3.141592653589793 upper=3.141592653589793 effort=1000.0 velocity=2.5
- joint wrist_roll_joint: limit lower=0 upper=0 effort=0 velocity=0 -> lower=-3.141592653589793 upper=3.141592653589793 effort=1000.0 velocity=2.5
- joint wrist_yaw_joint: limit lower=0 upper=0 effort=0 velocity=0 -> lower=-3.141592653589793 upper=3.141592653589793 effort=1000.0 velocity=2.5
