Commit message: added proper joint movement

File: src/2000-SimplifiedAssembly-06/urdf/ros2_drive_urdf.xacro (robot description, xacro)
@@ -35,5 +35,5 @@
     <parent link="chassis" />
     <child link="Left_Suspension" />
-    <axis xyz="0 0 0" />
+    <axis xyz="0 0 1" />
     <visual>
       <material name="silver" >
@@ -64,5 +64,5 @@
     <parent link="Left_Suspension" />
     <child link="Left_Rocker2Bogey" />
-    <axis xyz="0 0 0" />
+    <axis xyz="0 0 1" />
   </joint>
   <link name="Left_FrontWheel">
@@ -81,9 +81,9 @@
     </visual>
     </link>
-  <joint name="Left_FrontMotor" type="fixed">
+  <joint name="Left_FrontMotor" type="continuous">
     <origin xyz="0.420116653006438 -0.311178663383762 -0.321965022741944" rpy="-3.10907021451776 0.142647279967552 -2.62794863504613" />
     <parent link="Left_Rocker2Bogey" />
     <child link="Left_FrontWheel" />
-    <axis xyz="0 0 0" />
+    <axis xyz="0 0 1" />
   </joint>
   <link name="Left_MiddleWheel">
@@ -102,9 +102,9 @@
     </visual>
     </link>
-  <joint name="Left_MiddleMotor" type="fixed">
+  <joint name="Left_MiddleMotor" type="continuous">
     <origin xyz="-0.0377496814532355 -0.221089089566748 -0.382855126553232" rpy="2.99569987669468 0.0107184424391394 1.9322821944261" />
     <parent link="Left_Rocker2Bogey" />
     <child link="Left_MiddleWheel" />
-    <axis xyz="0 0 0" />
+    <axis xyz="0 0 1" />
   </joint>
   <link name="Left_BackWheel">
@@ -123,9 +123,9 @@
     </visual>
     </link>
-  <joint name="Left_BackMotor" type="fixed">
+  <joint name="Left_BackMotor" type="continuous">
     <origin xyz="-0.34870017734109 -0.0329830956324644 -0.41538946795221" rpy="-3.14159265358979 0 2.21631381188862" />
     <parent link="Left_Suspension" />
     <child link="Left_BackWheel" />
-    <axis xyz="0 0 0" />
+    <axis xyz="0 0 1" />
   </joint>
   <link name="Right_Suspension">
@@ -148,5 +148,5 @@
     <parent link="chassis" />
     <child link="Right_Suspension" />
-    <axis xyz="0 0 0" />
+    <axis xyz="0 0 1" />
   </joint>
   <link name="Right_Rocker2Bogey">
@@ -169,5 +169,5 @@
     <parent link="Right_Suspension" />
     <child link="Right_Rocker2Bogey" />
-    <axis xyz="0 0 0" />
+    <axis xyz="0 0 1" />
   </joint>
   <link name="Right_FrontWheel">
@@ -186,9 +186,9 @@
     </visual>
     </link>
-  <joint name="Right_FrontMotor" type="fixed">
+  <joint name="Right_FrontMotor" type="continuous">
     <origin xyz="0.420116653006444 -0.31117866338377 0.321965022741935" rpy="3.10907021451775 -0.142647279967552 -2.62794863504613" />
     <parent link="Right_Rocker2Bogey" />
     <child link="Right_FrontWheel" />
-    <axis xyz="0 0 0" />
+    <axis xyz="0 0 1" />
   </joint>
   <link name="Right_MiddleWheel">
@@ -207,9 +207,9 @@
     </visual>
     </link>
-  <joint name="Right_MiddleMotor" type="fixed">
+  <joint name="Right_MiddleMotor" type="continuous">
     <origin xyz="-0.037749681453219 -0.22108908956674 0.382855126553235" rpy="-2.99569987669466 -0.0107184424391394 1.9322821944261" />
     <parent link="Right_Rocker2Bogey" />
     <child link="Right_MiddleWheel" />
-    <axis xyz="0 0 0" />
+    <axis xyz="0 0 1" />
   </joint>
   <link name="Right_BackWheel">
@@ -228,9 +228,9 @@
     </visual>
     </link>
-  <joint name="Right_BackMotor" type="fixed">
+  <joint name="Right_BackMotor" type="continuous">
     <origin xyz="-0.348700177341093 -0.0329830956324626 0.415389467952218" rpy="-3.14159265358979 0 2.21631381188862" />
     <parent link="Right_Suspension" />
     <child link="Right_BackWheel" />
-    <axis xyz="0 0 0" />
+    <axis xyz="0 0 1" />
   </joint>
 </robot>

Commit message: initial ros workings

File: src/2000-SimplifiedAssembly-06/urdf/ros2_drive_urdf.xacro (robot description, xacro)
@@ -15,4 +15,9 @@
       </geometry>
     </visual>
+    <collision>
+      <geometry>
+        <mesh filename="package://2000-SimplifiedAssembly-06/meshes/visual/chassis.STL" scale="1 1 1"/>
+      </geometry>
+    </collision>
     </link>
   <link name="Left_Suspension">
@@ -30,4 +35,9 @@
       </geometry>
     </visual>
+    <collision>
+      <geometry>
+        <mesh filename="package://2000-SimplifiedAssembly-06/meshes/visual/Left_Suspension.STL" scale="1 1 1"/>
+      </geometry>
+    </collision>
     </link>
   <joint name="Left_Rocker" type="fixed">
@@ -59,4 +69,9 @@
       </geometry>
     </visual>
+    <collision>
+      <geometry>
+        <mesh filename="package://2000-SimplifiedAssembly-06/meshes/visual/Left_Rocker2Bogey.STL" scale="1 1 1"/>
+      </geometry>
+    </collision>
     </link>
   <joint name="Left_Bogey" type="fixed">
@@ -80,4 +95,9 @@
       </geometry>
     </visual>
+    <collision>
+      <geometry>
+        <mesh filename="package://2000-SimplifiedAssembly-06/meshes/visual/Left_FrontWheel.STL" scale="1 1 1"/>
+      </geometry>
+    </collision>
     </link>
   <joint name="Left_FrontMotor" type="continuous">
@@ -101,4 +121,9 @@
       </geometry>
     </visual>
+    <collision>
+      <geometry>
+        <mesh filename="package://2000-SimplifiedAssembly-06/meshes/visual/Left_MiddleWheel.STL" scale="1 1 1"/>
+      </geometry>
+    </collision>
     </link>
   <joint name="Left_MiddleMotor" type="continuous">
@@ -122,4 +147,9 @@
       </geometry>
     </visual>
+    <collision>
+      <geometry>
+        <mesh filename="package://2000-SimplifiedAssembly-06/meshes/visual/Left_BackWheel.STL" scale="1 1 1"/>
+      </geometry>
+    </collision>
     </link>
   <joint name="Left_BackMotor" type="continuous">
@@ -143,4 +173,9 @@
       </geometry>
     </visual>
+    <collision>
+      <geometry>
+        <mesh filename="package://2000-SimplifiedAssembly-06/meshes/visual/Right_Suspension.STL" scale="1 1 1"/>
+      </geometry>
+    </collision>
     </link>
   <joint name="Right_Rocker" type="fixed">
@@ -164,4 +199,9 @@
       </geometry>
     </visual>
+    <collision>
+      <geometry>
+        <mesh filename="package://2000-SimplifiedAssembly-06/meshes/visual/Right_Rocker2Bogey.STL" scale="1 1 1"/>
+      </geometry>
+    </collision>
     </link>
   <joint name="Right_Bogey" type="fixed">
@@ -185,4 +225,9 @@
       </geometry>
     </visual>
+    <collision>
+      <geometry>
+        <mesh filename="package://2000-SimplifiedAssembly-06/meshes/visual/Right_FrontWheel.STL" scale="1 1 1"/>
+      </geometry>
+    </collision>
     </link>
   <joint name="Right_FrontMotor" type="continuous">
@@ -206,4 +251,9 @@
       </geometry>
     </visual>
+    <collision>
+      <geometry>
+        <mesh filename="package://2000-SimplifiedAssembly-06/meshes/visual/Right_BackWheel.STL" scale="1 1 1"/>
+      </geometry>
+    </collision>
     </link>
   <joint name="Right_MiddleMotor" type="continuous">
@@ -227,4 +277,9 @@
       </geometry>
     </visual>
+    <collision>
+      <geometry>
+        <mesh filename="package://2000-SimplifiedAssembly-06/meshes/visual/Right_BackWheel.STL" scale="1 1 1"/>
+      </geometry>
+    </collision>
     </link>
   <joint name="Right_BackMotor" type="continuous">
@@ -234,3 +289,9 @@
     <axis xyz="0 0 1" />
   </joint>
+  <gazebo>
+    <!-- Joint state publisher -->
+    <plugin filename="gz_ros2_control-system" name="gz_ros2_control::GazeboSimROS2ControlPlugin">
+      <parameters>$(find diff_drive)/config/diffbot_controllers.yaml</parameters>
+    </plugin>
+  </gazebo>
 </robot>

File: src/diff_drive/ros2_control/diffbot.ros2_control.xacro (robot description, xacro)
@@ -16,10 +16,30 @@
         </hardware>
       </xacro:if>
-      <joint name="${prefix}left_wheel_joint">
+      <joint name="Left_FrontMotor">
         <command_interface name="velocity"/>
         <state_interface name="position"/>
         <state_interface name="velocity"/>
       </joint>
-      <joint name="${prefix}right_wheel_joint">
+      <joint name="Left_MiddleMotor">
+        <command_interface name="velocity"/>
+        <state_interface name="position"/>
+        <state_interface name="velocity"/>
+      </joint>
+      <joint name="Left_BackMotor">
+        <command_interface name="velocity"/>
+        <state_interface name="position"/>
+        <state_interface name="velocity"/>
+      </joint>
+      <joint name="Right_FrontMotor">
+        <command_interface name="velocity"/>
+        <state_interface name="position"/>
+        <state_interface name="velocity"/>
+      </joint>
+      <joint name="Right_MiddleMotor">
+        <command_interface name="velocity"/>
+        <state_interface name="position"/>
+        <state_interface name="velocity"/>
+      </joint>
+      <joint name="Right_BackMotor">
         <command_interface name="velocity"/>
         <state_interface name="position"/>
